Commit message: Simulation

File: WasteClassification/scara.urdf (robot description, URDF)
Before this commit: robot scara, 4 links, 3 joints
Links:
- link end_effector: geometry visual cylinder length=0.1 radius=0.02
- link link1: geometry visual box size=0.5 0.05 0.05
- link link2: geometry visual box size=0.4 0.05 0.05
Joints:
- joint joint1: limit lower=-3.14 upper=3.14 effort=100 velocity=1.0 -> lower=-3.14 upper=3.14 effort=10 velocity=1.0; origin (none) -> xyz=0 0 0.1 rpy=0 0 0
- joint joint2: limit lower=-3.14 upper=3.14 effort=100 velocity=1.0 -> lower=-3.14 upper=3.14 effort=10 velocity=1.0; origin (none) -> xyz=0.5 0 0 rpy=0 0 0
- joint joint3: limit lower=0 upper=0.2 effort=50 velocity=0.5 -> lower=-0.2 upper=0.2 effort=10 velocity=0.1; origin (none) -> xyz=0.4 0 0 rpy=0 0 0

Commit message: fixed sim

File: WasteClassification/scara.urdf (robot description, URDF)
Before this commit: robot scara, 4 links, 3 joints
Joints:
- joint joint1: origin xyz=0 0 0.1 rpy=0 0 0 -> xyz=0 0 0.3 rpy=0 0 0

Commit message: improved pybullet simulation

File: WasteClassification/scara.urdf (robot description, URDF)
Before this commit: robot scara, 4 links, 3 joints
Links:
- added link world
- link base: mass None -> 1.0; geometry collision box size=0.1 0.1 0.02
- link end_effector: mass None -> 0.1; geometry collision cylinder length=0.1 radius=0.02; visual cylinder length=0.1 radius=0.02
- link link1: mass None -> 0.5; geometry collision box size=0.5 0.05 0.05; visual box size=0.5 0.05 0.05
- link link2: mass None -> 0.4; geometry collision box size=0.4 0.05 0.05; visual box size=0.4 0.05 0.05
Joints:
- added joint base_x_slider: type prismatic, parent world, child base, origin xyz=0 0 0 rpy=0 0 0, axis 1 0 0, limit lower=-1.0 upper=4.0 effort=100 velocity=0.5

Commit message: improved simulation

File: WasteClassification/scara.urdf (robot description, URDF)
Before this commit: robot scara, 5 links, 4 joints
Links:
- link base: geometry collision box size=0.1 0.1 0.02; visual box size=0.1 0.1 0.02
